Commit message: modify arx5go2.urdf 1

File: resources/robots/go2/urdf/arx5go2.urdf (robot description, URDF)
Before this commit: robot go2_description, 37 links, 36 joints
Joints:
- joint zarx5p2_mount: origin xyz=0.0 0 0.057 rpy=0 0 0 -> xyz=0.1934 0 0.057 rpy=0 0 0

Commit message: Revert "modify arx5go2.urdf 1"
This reverts commit 435dba104bbf084342a70cc705b53eb13841c316.

File: resources/robots/go2/urdf/arx5go2.urdf (robot description, URDF)
Before this commit: robot go2_description, 37 links, 36 joints
Joints:
- joint zarx5p2_mount: origin xyz=0.1934 0 0.057 rpy=0 0 0 -> xyz=0.0 0 0.057 rpy=0 0 0
